File: Encoder/Encoder.kicad_sch (KiCad schematic)
At the start: 117 parts, among them J1 Conn_01x02_Socket, J2 Conn_01x02_Socket, J3 Conn_01x04_Socket, U1 TL072, U2 TL072, U3 TL072, U4 TL072, U5 MC1496, U6 NE5532, U7 TL072, U8 NE5532, U9 TL072

Commit message: new board layout
Parts:
- added TP_GND5, TP_L2: TestPoint, TestPoint:TestPoint_Pad_D1.5mm, symbol Connector:TestPoint
- added unit 3 of U8
- added unit 3 of U9
- renumbered U2 to U1, U3 to U2, U1 to U3
Connections:
- net +9V: now also U8.8 (V+), U9.8 (V+); no longer U8.8 (V+), U9.8 (V+)
- net -9V: now also U8.4 (V-), U9.4 (V-); no longer U8.4 (V-), U9.4 (V-)
- net GND: now also TP_GND5.1
- net right: now also U3.3 (+); no longer U3.5 (+)
- net at C14.2, R11.1: now also U3.6 (-), U3.7; no longer U3.1, U3.2 (-)
- net at C11.2, R8.2: now also U1.5 (+); no longer U1.3 (+)
- net at C17.2, R12.2: now also U2.3 (+); no longer U2.5 (+)
- net at C18.2, R14.1, R35.1: now also U2.1, U2.2 (-); no longer U2.6 (-), U2.7
- net at C16.2, R13.1, R34.1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: now also TP_L2.1
- net at C12.2, R9.1: now also U1.6 (-), U1.7; no longer U1.1, U1.2 (-)
- net at C13.2, R6.2: now also U3.5 (+); no longer U3.3 (+)
- new net: R5.1, U3.1, U3.2 (-)
- no-connect marks 1 -> 3
Changed lines of the file:
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@@
 	)
 	(junction
+		(at 196.85 83.82)
+		(diameter 0)
+		(color 0 0 0 0)
+	)
+	(junction
 		(at 195.58 83.82)
 		(diameter 0)
@@
 	)
 	(junction
+		(at 166.37 91.44)
+		(diameter 0)
+		(color 0 0 0 0)
+	)
+	(junction
 		(at 100.33 369.57)
 		(diameter 0)
@@
 	)
 	(no_connect
+		(at 392.43 113.03)
+	)
+	(no_connect
+		(at 318.77 77.47)
+	)
+	(no_connect
 		(at 20.32 95.25)
 	)
@@
 	(wire
 		(pts
+			(xy 196.85 90.17) (xy 196.85 83.82)
+		)
+		(stroke
+			(width 0)
+			(type default)
+		)
+	)
+	(wire
+		(pts
 			(xy 81.28 105.41) (xy 81.28 106.68)
 		)
@@
 		(shape input)
 		(at 43.18 400.05 0)
-		(fields_autoplaced yes)
 		(effects
 			(font
@@
 		)
 		(property "Intersheetrefs" "${INTERSHEET_REFS}"
-			(at 50.0357 400.05 0)
+			(at 53.8457 392.43 0)
 			(hide yes)
 			(show_name no)
@@
 	)
 	(symbol
+		(lib_id "Connector:TestPoint")
+		(at 166.37 91.44 270)
+		(unit 1)
+		(body_style 1)
+		(exclude_from_sim no)
+		(in_bom yes)
+		(on_board yes)
+		(in_pos_files yes)
+		(dnp no)
+		(fields_autoplaced yes)
+		(property "Reference" "TP_GND5"
+			(at 171.45 90.1699 90)
+			(show_name no)
+			(do_not_autoplace no)
+			(effects
+				(font
+					(size 1.27 1.27)
+				)
+				(justify left)
+			)
+		)
+		(property "Value" "TestPoint"
+			(at 171.45 92.7099 90)
+			(show_name no)
+			(do_not_autoplace no)
+			(effects
+				(font
+					(size 1.27 1.27)
+				)
+				(justify left)
+			)
+		)
+		(property "Footprint" "TestPoint:TestPoint_Pad_D1.5mm"
+			(at 166.37 96.52 0)
+			(hide yes)
+			(show_name no)
+			(do_not_autoplace no)
+			(effects
+				(font
+					(size 1.27 1.27)
+				)
+			)
+		)
+		(property "Datasheet" ""
+			(at 166.37 96.52 0)
+			(hide yes)
+			(show_name no)
+			(do_not_autoplace no)
+			(effects
+				(font
+					(size 1.27 1.27)
+				)
+			)
+		)
+		(property "Description" "test point"
+			(at 166.37 91.44 0)
+			(hide yes)
+			(show_name no)
+			(do_not_autoplace no)
+			(effects
+				(font
+					(size 1.27 1.27)
+				)
+			)
+		)
+		(pin "1"
+		)
+		(instances
+			(project "Encoder"
+				(path "/dd383f0c-7a62-48d5-8ebf-05a2096c9cf7"
+					(reference "TP_GND5")
+					(unit 1)
+				)
+			)
+		)
+	)
+	(symbol
 		(lib_id "Device:R_US")
 		(at 265.43 92.71 90)
@@
 		(lib_id "Amplifier_Operational:TL072")
 		(at 189.23 113.03 0)
-		(unit 2)
+		(unit 1)
 		(body_style 1)
 		(exclude_from_sim no)
@@
 		(dnp no)
 		(fields_autoplaced yes)
-		(property "Reference" "U3"
+		(property "Reference" "U2"
 			(at 189.23 102.87 0)
 			(show_name no)
@@
 			(project "Encoder"
 				(path "/dd383f0c-7a62-48d5-8ebf-05a2096c9cf7"
-					(reference "U3")
-					(unit 2)
+					(reference "U2")
+					(unit 1)
 				)
 			)
@@
 	)
 	(symbol
+		(lib_id "Connector:TestPoint")
+		(at 196.85 90.17 180)
+		(unit 1)
+		(body_style 1)
+		(exclude_from_sim no)
+		(in_bom yes)
+		(on_board yes)
+		(in_pos_files yes)
+		(dnp no)
+		(fields_autoplaced yes)
+		(property "Reference" "TP_L2"
+			(at 199.39 92.2019 0)
+			(show_name no)
+			(do_not_autoplace no)
+			(effects
+				(font
+					(size 1.27 1.27)
+				)
+				(justify right)
+			)
+		)
+		(property "Value" "TestPoint"
+			(at 199.39 94.7419 0)
+			(show_name no)
+			(do_not_autoplace no)
+			(effects
+				(font
+					(size 1.27 1.27)
+				)
+				(justify right)
+			)
+		)
+		(property "Footprint" "TestPoint:TestPoint_Pad_D1.5mm"
+			(at 191.77 90.17 0)
+			(hide yes)
+			(show_name no)
+			(do_not_autoplace no)
+			(effects
+				(font
+					(size 1.27 1.27)
+				)
+			)
+		)
+		(property "Datasheet" ""
+			(at 191.77 90.17 0)
+			(hide yes)
+			(show_name no)
+			(do_not_autoplace no)
+			(effects
+				(font
+					(size 1.27 1.27)
+				)
+			)
+		)
+		(property "Description" "test point"
+			(at 196.85 90.17 0)
+			(hide yes)
+			(show_name no)
+			(do_not_autoplace no)
+			(effects
+				(font
+					(size 1.27 1.27)
+				)
+			)
+		)
+		(pin "1"
+		)
+		(instances
+			(project "Encoder"
+				(path "/dd383f0c-7a62-48d5-8ebf-05a2096c9cf7"
+					(reference "TP_L2")
+					(unit 1)
+				)
+			)
+		)
+	)
+	(symbol
 		(lib_id "Device:R_US")
 		(at 203.2 113.03 90)
@@
 		(lib_id "Amplifier_Operational:TL072")
 		(at 138.43 81.28 0)
-		(unit 1)
+		(unit 2)
 		(body_style 1)
 		(exclude_from_sim no)
@@
 		(dnp no)
 		(fields_autoplaced yes)
-		(property "Reference" "U2"
+		(property "Reference" "U1"
 			(at 138.43 71.12 0)
 			(show_name no)
@@
 			(project "Encoder"
 				(path "/dd383f0c-7a62-48d5-8ebf-05a2096c9cf7"
-					(reference "U2")
-					(unit 1)
+					(reference "U1")
+					(unit 2)
 				)
 			)
@@
 		(lib_id "Amplifier_Operational:TL072")
 		(at 146.05 110.49 0)
-		(unit 1)
+		(unit 2)
 		(body_style 1)
 		(exclude_from_sim no)
@@
 				(path "/dd383f0c-7a62-48d5-8ebf-05a2096c9cf7"
 					(reference "U3")
-					(unit 1)
+					(unit 2)
 				)
 			)
@@
 		(lib_id "Amplifier_Operational:TL072")
 		(at 107.95 107.95 0)
-		(unit 2)
+		(unit 1)
 		(body_style 1)
 		(exclude_from_sim no)
@@
 		(dnp no)
 		(fields_autoplaced yes)
-		(property "Reference" "U1"
+		(property "Reference" "U3"
 			(at 107.95 97.79 0)
 			(show_name no)
@@
 			(project "Encoder"
 				(path "/dd383f0c-7a62-48d5-8ebf-05a2096c9cf7"
-					(reference "U1")
-					(unit 2)
+					(reference "U3")
+					(unit 1)
 				)
 			)

Commit message: encoder pcb test 1 is almost done
Parts:
- renumbered C5 to C1, C6 to C11, C4 to C12, C19 to C13, C20 to C14, C21 to C15, C22 to C16, C34 to C17, C26 to C18, C25 to C19, C3 to C2, C35 to C20, C30 to C21, C31 to C22, C11 to C23, C12 to C24, C13 to C25, C14 to C26, C38 to C27, C41 to C28, C39 to C29, C2 to C3, C40 to C30, C15 to C31, C16 to C32, C17 to C33, C18 to C34, C36 to C35, C37 to C36, C27 to C37, C24 to C38, C28 to C39, C1 to C4, C23 to C40, C29 to C41, C32 to C5, C33 to C6, D2 to D1, D1 to D2, D5 to D3, D6 to D4, D3 to D5, D4 to D6, J2 to J1, J1 to J2, R40 to R1, R5 to R10, R8 to R11, R6 to R12, R9 to R13, R10 to R14, R11 to R15, R43 to R16, R12 to R17, R44 to R18, R13 to R19, R3 to R2, R14 to R20, R15 to R21, R34 to R22, R35 to R23, R16 to R24, R36 to R25, R17 to R26, R37 to R27, R18 to R28, R20 to R29, R1 to R3, R38 to R30, R21 to R31, R19 to R32, R22 to R33, R23 to R34, R29 to R35, R24 to R36, R31 to R37, R30 to R38, R26 to R39, R25 to R40, R32 to R41, R33 to R42, R27 to R43, R28 to R44, R39 to R5, R2 to R6, R41 to R7, R42 to R8, R7 to R9, U6 to U10, U8 to U10, U8 to U2, U6 to U2, U2 to U3, U3 to U4, U2 to U4, U4 to U5, U7 to U6, U9 to U8, U5 to U9
Connections:
- net GND: now also U8.3 (+), U8.5 (+); no longer U8.3 (+), U8.5 (+)
- net at R45.2, R46.2, R47.2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: now also U8.6 (-); no longer U8.2 (-)
- net at R48.2, R49.1: now also U8.7; no longer U8.1
- net at R49.2, R50.1: now also U8.2 (-); no longer U8.6 (-)
- net at R1.1, R50.2: now also U8.1; no longer U8.7
