File: Encoder/Encoder_compact.kicad_sch (KiCad schematic)
At the start: 120 parts, among them J1 Conn_01x02_Socket, J2 Conn_01x02_Socket, J3 Conn_01x04_Socket, U1 TL072, U2 TL072, U3 TL072, U4 TL072, U5 MC1496, U6 NE5532, U7 TL072, U8 NE5532, U9 TL072

Commit message: 2 versions are available right now need to test the actual footprint before starting -- the 19k and 38k are still missing
Parts:
- removed JP1: Jumper_0R, Resistor_THT:R_Axial_DIN0207_L6.3mm_D2.5mm_P7.62mm_Horizontal, symbol R0:Jumper_0R
- added C42, C43, C44: 100n, Capacitor_THT:C_Disc_D5.0mm_W2.5mm_P5.00mm, symbol Device:C_US
- added J4: Conn_01x04_Socket, Connector_PinSocket_2.54mm:PinSocket_1x04_P2.54mm_Vertical, symbol Connector:Conn_01x04_Socket
- added TP11: 19K_IN, TestPoint:TestPoint_Pad_D1.5mm, symbol Connector:TestPoint
- added TP12: 38K_IN, TestPoint:TestPoint_Pad_D1.5mm, symbol Connector:TestPoint
- added TP13: U1A_OUT, TestPoint:TestPoint_Pad_D1.5mm, symbol Connector:TestPoint
- added TP14: U3A_OUT, TestPoint:TestPoint_Pad_D1.5mm, symbol Connector:TestPoint
- added TP15: U1B_OUT, TestPoint:TestPoint_Pad_D1.5mm, symbol Connector:TestPoint
- added TP16: U3B_OUT, TestPoint:TestPoint_Pad_D1.5mm, symbol Connector:TestPoint
- added TP17: U4A_OUT, TestPoint:TestPoint_Pad_D1.5mm, symbol Connector:TestPoint
- added TP18: U5A_OUT, TestPoint:TestPoint_Pad_D1.5mm, symbol Connector:TestPoint
- added TP19: U5B_OUT, TestPoint:TestPoint_Pad_D1.5mm, symbol Connector:TestPoint
- added TP20: U6A_OUT, TestPoint:TestPoint_Pad_D1.5mm, symbol Connector:TestPoint
- added TP21: U6B_OUT, TestPoint:TestPoint_Pad_D1.5mm, symbol Connector:TestPoint
- added TP22: MOD_OUT_P, TestPoint:TestPoint_Pad_D1.5mm, symbol Connector:TestPoint
- added TP23: MOD_OUT_N, TestPoint:TestPoint_Pad_D1.5mm, symbol Connector:TestPoint
- added TP24: U10A_OUT, TestPoint:TestPoint_Pad_D1.5mm, symbol Connector:TestPoint
- added TP25: U10B_OUT, TestPoint:TestPoint_Pad_D1.5mm, symbol Connector:TestPoint
- added TP26: U8A_OUT, TestPoint:TestPoint_Pad_D1.5mm, symbol Connector:TestPoint
- added TP27: U8B_OUT, TestPoint:TestPoint_Pad_D1.5mm, symbol Connector:TestPoint
- added TP28: U2A_OUT, TestPoint:TestPoint_Pad_D1.5mm, symbol Connector:TestPoint
- added TP29: OUT, TestPoint:TestPoint_Pad_D1.5mm, symbol Connector:TestPoint
- added TP30, TP31, TP32: GND, TestPoint:TestPoint_Pad_D1.5mm, symbol Connector:TestPoint
- renumbered C5 to C1, C6 to C11, C4 to C12, C19 to C13, C20 to C14, C21 to C15, C22 to C16, C34 to C17, C26 to C18, C25 to C19, C3 to C2, C35 to C20, C30 to C21, C31 to C22, C11 to C23, C12 to C24, C13 to C25, C14 to C26, C38 to C27, C41 to C28, C39 to C29, C2 to C3, C40 to C30, C15 to C31, C16 to C32, C17 to C33, C18 to C34, C36 to C35, C37 to C36, C27 to C37, C24 to C38, C28 to C39, C1 to C4, C23 to C40, C29 to C41, C32 to C5, C33 to C6, D2 to D1, D1 to D2, D5 to D3, D6 to D4, D3 to D5, D4 to D6, J2 to J1, J1 to J2, R40 to R1, R5 to R10, R8 to R11, R6 to R12, R9 to R13, R10 to R14, R11 to R15, R43 to R16, R12 to R17, R44 to R18, R13 to R19, R3 to R2, R14 to R20, R15 to R21, R34 to R22, R35 to R23, R16 to R24, R36 to R25, R17 to R26, R37 to R27, R18 to R28, R20 to R29, R1 to R3, R38 to R30, R21 to R31, R19 to R32, R22 to R33, R23 to R34, R29 to R35, R24 to R36, R31 to R37, R30 to R38, R26 to R39, R25 to R40, R32 to R41, R33 to R42, R27 to R43, R28 to R44, R39 to R5, R2 to R6, R41 to R7, R42 to R8, R7 to R9, U6 to U10, U8 to U10, U8 to U2, U6 to U2, U2 to U3, U3 to U4, U2 to U4, U4 to U5, U7 to U6, U9 to U8, U5 to U9
Connections:
- net +9V: now also C43.2
- net -9V: now also C42.2, C44.2
- net GND: now also U8.3 (+), U8.5 (+), C42.1, C43.1, C44.1, J4.4 (Pin_4), TP30.1, TP31.1, TP32.1; no longer U8.3 (+), U8.5 (+)
- net U2A_OUT: now reaches C17.2, R16.1, U2.1
- net U2A_OUT: now also U2.2 (-), TP28.1; no longer U2.3 (+)
- net at C20.2, R8.2: now also U2.3 (+); no longer U2.2 (-)
- net U3B_OUT: now reaches C26.2, R15.1, U3.6 (-), U3.7
- net U3B_OUT: now also TP16.1
- net U6A_OUT: now reaches R25.2, R27.1, U6.1
- net U6A_OUT: now also TP20.1
- net U3A_OUT: now reaches R10.1, U3.1, U3.2 (-)
- net U3A_OUT: now also TP14.1
- net U10B_OUT: now reaches C6.2, R7.1, U10.6 (-), U10.7
- net U10B_OUT: now also TP25.1
- net U5B_OUT: now reaches R28.2, R32.1, U5.7
- net U5B_OUT: now also TP19.1
- net U6B_OUT: now reaches R30.2, R45.1, U6.7
- net U6B_OUT: now also TP21.1
- net at R45.2, R46.2, R47.2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: now also U8.6 (-); no longer U8.2 (-)
- net U8B_OUT: now reaches R48.2, R49.1
- net U8B_OUT: now also U8.7, TP27.1; no longer U8.1
- net at R49.2, R50.1: now also U8.2 (-); no longer U8.6 (-)
- net U8A_OUT: now reaches R1.1, R50.2
- net U8A_OUT: now also U8.1, TP26.1; no longer U8.7
- net U5A_OUT: now reaches R24.2, R26.1, U5.1
- net U5A_OUT: now also TP18.1
- net U4A_OUT: now reaches C34.2, R20.1, R23.1, U4.1, U4.2 (-)
- net U4A_OUT: now also TP17.1
- net U10A_OUT: now reaches R44.2, R46.1, U10.1
- net U10A_OUT: now also TP24.1
- net U1B_OUT: now reaches C24.2, R13.1, U1.6 (-), U1.7
- net U1B_OUT: now also TP15.1
- net OUT: now reaches C35.2, U2.7
- net OUT: now also U2.6 (-), J4.1 (Pin_1), TP29.1; no longer U2.5 (+)
- net at C36.1, R18.2: now also U2.5 (+); no longer U2.6 (-)
- net MOD_OUT_N: now reaches C40.1, R36.2, U9.12 (VO-)
- net MOD_OUT_N: now also TP23.1
- net MOD_OUT_P: now reaches C38.1, R34.2, U9.6 (VO+)
- net MOD_OUT_P: now also TP22.1
- net U1A_OUT: now reaches R9.1, U1.1, U1.2 (-)
- net U1A_OUT: now also TP13.1
- net 19K_IN: now reaches R47.1
- net 19K_IN: now also TP11.1
- net 38K_IN: now reaches R38.2
- net 38K_IN: now also TP12.1
- no-connect marks 3 -> 5
Other:
- title: (none) -> FM Stereo Encoder
