File: Encoder/older versions/Encoder_compact.kicad_pcb (KiCad board)
At the start: 2 copper layers, 111 x 110 mm, 145 parts, among them J1 Conn_01x02_Socket, J2 Conn_01x02_Socket, J3 Conn_01x04_Socket, J4 Conn_01x04_Socket, U1 TL072, U10 NE5532, U2 NE5532, U3 TL072, U4 TL072, U5 TL072, U6 TL072, U8 TL072, U9 MC1496

Commit message: encoder V1 is done need testing
Other:
- board text removed: "Rev 1 2026-10-22"
Changed lines of the file:
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@@
 			(outputformat 1)
 			(mirror no)
-			(drillshape 1)
+			(drillshape 0)
 			(scaleselection 1)
-			(outputdirectory "")
+			(outputdirectory "../../../")
 		)
 	)
@@
 			)
 			(justify left)
-		)
-	)
-	(gr_text "Rev 1  2026-10-22"
-		(at 74.84 148.57 0)
-		(layer "F.SilkS")
-		(effects
-			(font
-				(size 1 1)
-				(thickness 0.15)
-			)
-			(justify left)
